Commit message: update-radar sensor removed
The radar sensor was removed but will be returning.

File: aimm_gazebo/worlds/example_course.world.xacro (robot description, xacro)
@@ -19,8 +19,19 @@
       </wind_objs>
     </xacro:usv_wind_gazebo>
+    <!-- The light buoy -->
+    <include>
+      <uri>model://robotx_light_buoy</uri>
+      <pose>-511 218 0.25 0 0 3.14</pose>
+    </include>
+    <!-- The VRX animal buoys -->
+    <include>
+      <name>platypus_buoy</name>
+      <pose>-512 170 0 0 0 0</pose>
+      <uri>model://platypus_buoy</uri>
+    </include>
     <!-- The obstacle course -->
     <include>
-      <uri>model://obstacle_course0</uri>
-      <pose>-560 170 0 0 0 -2.04</pose>
+      <uri>model://aimm_course</uri>
+      <pose>-460 300 0 0 0 -2</pose>
     </include>
   </world>

File: aimm_gazebo/worlds/gymkhana.world.xacro (robot description, xacro)
@@ -44,5 +44,5 @@
       <ready_state_duration>10</ready_state_duration>
       <running_state_duration>300</running_state_duration>
-      <!-- Per-plugin flag, different from env var AIMM_EXIT_ON_COMPLETION.
+      <!-- Per-plugin flag, different from env var VRX_EXIT_ON_COMPLETION.
            Respect top-level plugin finished status. -->
       <per_plugin_exit_on_completion>true</per_plugin_exit_on_completion>
@@ -57,5 +57,5 @@
       <task_name>gymkhana_channel</task_name>
       <task_info_topic>/aimm/gymkhana_channel/task/info</task_info_topic>
-      <contact_debug_topic>/lpv/gymkhana_channel/debug/contact</contact_debug_topic>
+      <contact_debug_topic>/aimm/gymkhana_channel/debug/contact</contact_debug_topic>
       <!-- Keep Gazebo running after this sub-task is completed -->
       <per_plugin_exit_on_completion>false</per_plugin_exit_on_completion>

File: aimm_gazebo/worlds/perception_task.world.xacro (robot description, xacro)
@@ -37,5 +37,5 @@
       <!-- Pose of each object is expressed relative to the body frame
            of the object named in the frame field - i.e., relative to
-           the lp-v-->
+           the wam-v-->
       <object_sequence>
         <object>

File: aimm_gazebo/worlds/sydneyregatta.world.xacro (robot description, xacro)
@@ -8,5 +8,5 @@
     <xacro:include filename="$(find wave_gazebo)/world_models/ocean_waves/model.xacro"/>
     <xacro:ocean_waves scale="2.5"/>
-    <!--Wind for the WAM-V. Note, wind parameters are set in the plug.-->
+    <!--Wind for the LPV-4. Note, wind parameters are set in the plug.-->
     <xacro:include filename="$(find aimm_gazebo)/worlds/xacros/usv_wind_plugin.xacro"/>
     <xacro:usv_wind_gazebo>

File: aimm_gazebo/worlds/sydneyregatta.xacro (robot description, xacro)
@@ -39,5 +39,5 @@
       <uri>model://sydney_regatta</uri>
     </include>
-    <!-- The posts for securing the WAM-V -->
+    <!-- The posts for securing the LPV-4 -->
     <include>
       <name>post_0</name>
@@ -55,5 +55,5 @@
       <uri>model://post</uri>
     </include>
-    <!-- Antenna for communication with the WAM-V -->
+    <!-- Antenna for communication with the LPV-4 -->
     <include>
       <pose>-531.063721 147.668579 1.59471 -0.068142 0 -0.1</pose>

File: aimm_gazebo/worlds/xacros/sandisland_minus_scene.xacro (robot description, xacro)
@@ -30,5 +30,5 @@
       <uri>model://sandisland</uri>
     </include>
-    <!-- The posts for securing the WAM-V -->
+    <!-- The posts for securing the LPV-4 -->
     <include>
       <name>post_0</name>
@@ -46,5 +46,5 @@
       <uri>model://post</uri>
     </include>
-    <!-- Antenna for communication with the WAM-V -->
+    <!-- Antenna for communication with the LPV-4 -->
     <include>
       <pose>175.69 114.29 1.37 0 0 2.00</pose>

File: aimm_gazebo/worlds/xacros/sydneyregatta_minus_scene.xacro (robot description, xacro)
@@ -30,5 +30,5 @@
       <uri>model://sydney_regatta</uri>
     </include>
-    <!-- The posts for securing the WAM-V -->
+    <!-- The posts for securing the LPV-4 -->
     <include>
       <name>post_0</name>
@@ -46,5 +46,5 @@
       <uri>model://post</uri>
     </include>
-    <!-- Antenna for communication with the WAM-V -->
+    <!-- Antenna for communication with the LPV-4 -->
     <include>
       <pose>-531.063721 147.668579 1.59471 -0.068142 0 -0.1</pose>

File: aimm_gazebo/worlds/xacros/usv_wind_plugin.xacro (robot description, xacro)
@@ -12,5 +12,5 @@
                          topic_wind_direction:=/aimm/debug/wind/direction
                          " >
-    <!--Gazebo Plugin for simulating WAM-V dynamics-->
+    <!--Gazebo Plugin for simulating LPV-4 dynamics-->
     <plugin name="wind" filename="libusv_gazebo_wind_plugin.so">
       <!-- models to be effected by the wind -->

File: lpv_description/urdf/battery.xacro (robot description, xacro)
@@ -4,7 +4,7 @@
     <link name="${namespace}/${prefix}_battery_link">
       <visual name="${prefix}_battery_visual">
-        <origin xyz="0 -1.03 -.45" rpy="0 0 0"/>
+        <origin xyz="0 -0.82 -.45" rpy="0 0 0"/>
         <geometry>
-          <mesh filename="package://aimm_gazebo/models/battery/mesh/battery.dae"/>
+          <mesh filename="package://aimm_gazebo/models/battery/mesh/battery.dae" scale=".8 .8 .8"/>
         </geometry>
       </visual>

File: lpv_description/urdf/lpv_base.urdf.xacro (robot description, xacro)
@@ -1,85 +1,7 @@
 <?xml version="1.0"?>
-<robot xmlns:xacro="http://ros.org/wiki/xacro" name="lpv-4">
+<robot xmlns:xacro="http://ros.org/wiki/xacro" name="LPV-4">
   <xacro:arg name="namespace" default="lpv"/>
   <xacro:property name="namespace" value="$(arg namespace)" scope="global" />
-  <xacro:macro name="main_collisions" params="prefix reflect:=1">
-    <!-- Main float
-    <collision name="${prefix}_float">
-      <origin xyz="-0.4 ${1.03*reflect} 0.2" rpy="${0*reflect} 1.57 0" />
-      <geometry>
-        <cylinder length="4" radius="0.2" />
-      </geometry>
-    </collision>
-    <collision name="${prefix}_mid_float">
-      <origin xyz="1.85 ${1.03*reflect} 0.3" rpy="${0*reflect} 1.38 0" />
-      <geometry>
-        <cylinder length="0.5" radius="0.17" />
-      </geometry>
-    </collision>
-    <collision name="${prefix}_front_float">
-      <origin xyz="2.3 ${1.03*reflect} 0.4" rpy="${0*reflect} 1.3 0" />
-      <geometry>
-        <cylinder length="0.45" radius="0.12" />
-      </geometry>
-    </collision>-->
-    <!-- Front beam
-    <collision name="front_${prefix}_beam_lower">
-      <origin xyz="0.9 ${0.85*reflect} 1" rpy="${0.78*reflect} 0 0" />
-      <geometry>
-        <cylinder length="0.5" radius="0.04" />
-      </geometry>
-    </collision>
-    <collision name="front_${prefix}_beam_upper">
-      <origin xyz="0.9 ${0.6*reflect} 1.18" rpy="${1.35*reflect} 0 0" />
-      <geometry>
-        <cylinder length="0.2" radius="0.04" />
-      </geometry>
-    </collision>-->
-    <!-- Mid beam
-    <collision name="mid_${prefix}_beam_lower">
-      <origin xyz="-0.65 ${0.99*reflect} 0.7" rpy="${0.1*reflect} 0.25 0" />
-      <geometry>
-        <cylinder length="0.45" radius="0.03" />
-      </geometry>
-    </collision>
-    <collision name="mid_${prefix}_beam_medium">
-      <origin xyz="-0.57 ${0.87*reflect} 1.05" rpy="${0.75*reflect} 0.25 0" />
-      <geometry>
-        <cylinder length="0.32" radius="0.03" />
-      </geometry>
-    </collision>
-    <collision name="mid_${prefix}_beam_upper">
-      <origin xyz="-0.55 ${0.65*reflect} 1.17" rpy="${1.35*reflect} 0.25 0" />
-      <geometry>
-        <cylinder length="0.3" radius="0.03" />
-      </geometry>
-    </collision>-->
-    <!-- Rear beam
-    <collision name="rear_${prefix}_beam_lower">
-      <origin xyz="-0.74 ${1.03*reflect} 0.7" rpy="${0*reflect} -0.15 0" />
-      <geometry>
-        <cylinder length="0.45" radius="0.03" />
-      </geometry>
-    </collision>
-    <collision name="rear_${prefix}_beam_medium">
-      <origin xyz="-0.79 ${0.91*reflect} 1.05" rpy="${0.75*reflect} -0.15 0" />
-      <geometry>
-        <cylinder length="0.32" radius="0.03" />
-      </geometry>
-    </collision>
-    <collision name="rear_${prefix}_beam_upper">
-      <origin xyz="-0.81 ${0.67*reflect} 1.18" rpy="${1.45*reflect} -0.15 0" />
-      <geometry>
-        <cylinder length="0.3" radius="0.03" />
-      </geometry>
-    </collision>-->
-    <!-- Joint
-    <collision name="${prefix}_joint">
-      <origin xyz="0.58 ${1.03*reflect} 0.6" rpy="${0*reflect} -0.6 0" />
-      <geometry>
-        <box size="0.65 0.2 0.1" />
-      </geometry>
-    </collision>-->
-  </xacro:macro>
+  <!-- base link -->
   <link name="${namespace}/base_link">
   </link>
@@ -89,32 +11,17 @@
   </joint>
   <link name="${namespace}/dummy_link">
-    <gazebo>
-      <plugin name="ground_truth_publisher" filename="libgazebo_ros_ground_truth_plugin.so">
-        <robotNamespace>$(arg namespace)</robotNamespace>
-        <updateRate>100</updateRate>
-        <bodyName>${namespace}/base_link</bodyName>
-        <topicName>ground_truth_pose</topicName>
-      </plugin>
-    </gazebo>
     <visual>
-      <origin xyz="0 -0 -0.6" rpy="0 0 0" />
+      <origin xyz="0 0 -0.5" rpy="0 0 3.14" />
       <geometry>
-        <mesh filename="package://lpv_description/models/LPV-Base/mesh/lpv_base.dae" scale="0.05 0.05 0.05"/>
+        <mesh filename="package://lpv_description/models/aimm-base/mesh/AIMMBoat.dae" scale="0.03 0.03 0.03"/>
       </geometry>
     </visual>
-    <collision>
+    <collision name="main_float">
+      <origin xyz="0 0 0.15" rpy="0 0 0" />
       <geometry>
-        <mesh filename="package://lpv_description/models/LPV-Base/mesh/lpv_base.dae" scale="0.05 0.05 0.05"/>
+        <box size="4.1 1.2 0.5"/>
       </geometry>
     </collision>
-     <!-- Top base
-    <collision name="top_base">
-      <origin xyz="0 -0 0.1" rpy="0 0 0" />
-      <geometry>
-        <box size="1 1 0.1" />
-      </geometry>
-    </collision>-->
     <inertial>
-      <!-- From WAM-V spec sheet -->
       <mass value="180.0"/>
       <inertia ixx="120.0" ixy="0.0" ixz="0.0" iyy="393" iyz="0.0" izz="446.0"/>

File: lpv_description/urdf/thrusters/engine.xacro (robot description, xacro)
@@ -1,4 +1,4 @@
 <?xml version="1.0"?>
-<robot xmlns:xacro="http://ros.org/wiki/xacro" name="wam-v-two-engines">
+<robot xmlns:xacro="http://ros.org/wiki/xacro" name="lpv-4-one-engine">
   <!-- Macro for inserting an engine with its propeller. -->
   <xacro:macro name="engine" params="prefix position:='0 0 0' orientation:='0 0 0'">
@@ -43,11 +43,13 @@
       </inertial>
     </link>
+    <!-- Revolute joint for yaw control (chasis to engine) -->
     <joint name="${namespace}/${prefix}_chasis_engine_joint" type="revolute">
       <axis xyz="0 0 1"/>
-      <limit lower="${-pi}" upper="${pi}" effort="10" velocity="10"/>
+      <limit lower="${-pi/2}" upper="${pi/2}" effort="20" velocity="20"/>
       <origin xyz="${position}" rpy="${orientation}"/>
       <parent link="${namespace}/base_link"/>
       <child link="${namespace}/${prefix}_engine_link"/>
     </joint>
+    <!-- Continuous joint for propeller rotation -->
     <joint name="${namespace}/${prefix}_engine_propeller_joint" type="continuous">
       <axis rpy="0 0 0" xyz="1 0 0"/>
@@ -58,4 +60,14 @@
       <dynamics friction="0.05" damping="0.05" />
     </joint>
+    <!-- Transmission for yaw control joint (chasis_engine_joint) -->
+    <transmission name="${namespace}/${prefix}_chasis_engine_joint_trans">
+      <type>transmission_interface/SimpleTransmission</type>
+      <joint name="${namespace}/${prefix}_chasis_engine_joint">
+        <hardwareInterface>EffortJointInterface</hardwareInterface>
+      </joint>
+      <actuator name="${namespace}/${prefix}_chasis_engine_actuator">
+        <mechanicalReduction>1</mechanicalReduction>
+      </actuator>
+    </transmission>
   </xacro:macro>
 </robot>

File: lpv_gazebo/urdf/components/lpv_camera.xacro (robot description, xacro)
@@ -1,5 +1,5 @@
 <?xml version="1.0"?>
 <robot xmlns:xacro="http://ros.org/wiki/xacro">
-  <xacro:macro name="lpv_camera" params="name x:=0.5 y:=0 z:=1.5 post_z_from:=1.2965 R:=0 P:=0 Y:=0 post_Y:=0 visualize:=False">
+  <xacro:macro name="lpv_camera" params="name x:=0.5 y:=0 z:=0 post_z_from:=0.35 R:=0 P:=0 Y:=0 post_Y:=0 visualize:=False">
     <!-- Define length variables for link positioning -->
     <xacro:property name="platform_z" value="${post_z_from}"/>
@@ -12,5 +12,5 @@
         <origin xyz="-0.033 0 0" rpy="0 0 ${pi/2}"/>
         <geometry>
-          <mesh filename="package://lpv_gazebo/models/mono_camera/mesh/mono_camera.dae"/>
+          <mesh filename="package://aimm_gazebo/models/mono_camera/mesh/mono_camera.dae"/>
         </geometry>
       </visual>

File: lpv_gazebo/urdf/components/lpv_gps.xacro (robot description, xacro)
@@ -1,5 +1,5 @@
 <?xml version="1.0" encoding="UTF-8"?>
 <robot xmlns:xacro="http://ros.org/wiki/xacro">
-  <xacro:macro name="lpv_gps" params="name:=gps x:=0.3 y:=0 z:=0.9
+  <xacro:macro name="lpv_gps" params="name:=gps x:=0.3 y:=0 z:=1.3
 				       R:=0 P:=0 Y:=0 update_rate:=15">
     <link name="${namespace}/${name}_link">

File: lpv_gazebo/urdf/dynamics/lpv_gazebo_dynamics_plugin.xacro (robot description, xacro)
@@ -1,6 +1,6 @@
 <?xml version="1.0"?>
 <robot xmlns:xacro="http://ros.org/wiki/xacro">
-  <xacro:macro name="usv_dynamics_gazebo" params="name width:=2.9 length:=4.9">
-    <!--Gazebo Plugin for simulating WAM-V dynamics-->
+  <xacro:macro name="usv_dynamics_gazebo" params="name width:=2.4 length:=4.9">
+    <!--Gazebo Plugin for simulating LPV-4 dynamics-->
     <gazebo>
       <plugin name="usv_dynamics_${name}" filename="libusv_gazebo_dynamics_plugin.so">

File: lpv_gazebo/urdf/lpv_gazebo.urdf.xacro (robot description, xacro)
@@ -1,8 +1,8 @@
 <?xml version="1.0"?>
-<!-- Basic WAM-V with gazebo plugins for dynamics -->
+<!-- Basic LPV-4 with gazebo plugins for dynamics -->
 <robot xmlns:xacro="http://ros.org/wiki/xacro"
-       name="lpv-4">
+       name="LPV-4">
   <xacro:arg name="locked" default="false" />
-  <xacro:arg name="thruster_config" default="H" />
+  <xacro:arg name="thruster_config" default="Z" />
   <xacro:arg name="camera_enabled" default="false" />
   <xacro:arg name="gps_enabled" default="false" />
@@ -33,6 +33,10 @@
   <xacro:arg name="yaml_thruster_generation" default="false"/>
   <xacro:arg name="thruster_xacro_file" default = ""/>
-  <!-- === The LP-V platform === -->
+  <!-- === The LPV-4 platform === -->
   <xacro:include filename="$(find lpv_gazebo)/urdf/lpv_gazebo.xacro"/>
+  <!-- === Batteries === -->
+  <xacro:include filename="$(find lpv_description)/urdf/battery.xacro"/>
+  <xacro:battery prefix="mid" position="-1.5 0 0.2" orientation="0 0 0"/>
+  <!--xacro:battery prefix="right" position="-2 -0.1 0.45" orientation="0 0 0 "/-->
   <!-- === Thrusters === -->
   <!-- Use thruster yaml file if given -->
@@ -43,5 +47,5 @@
   <xacro:unless value="$(arg yaml_thruster_generation)">
     <xacro:property name="thruster_conf" value="$(arg thruster_config)"/>
-    <!-- Default WAM-V with two aft thrusters -->
+    <!-- Default LPV-4 with two aft thrusters -->
     <xacro:if value="${thruster_conf == 'H'}">
        <xacro:lpv_gazebo thruster_layout="$(find lpv_gazebo)/urdf/thruster_layouts/lpv_aft_thrusters.xacro"/>
@@ -55,32 +59,8 @@
       <xacro:lpv_gazebo thruster_layout="$(find lpv_gazebo)/urdf/thruster_layouts/lpv_x_thrusters.xacro"/>
     </xacro:if>
+  <xacro:if value="${thruster_conf == 'Z'}">
+      <xacro:lpv_gazebo thruster_layout="$(find lpv_gazebo)/urdf/thruster_layouts/lpv_z_thrusters.xacro"/>
+    </xacro:if>
   </xacro:unless>
-  <!-- === Decide if we lock the robot to the world === -->
-  <xacro:if value="$(arg locked)">
-    <gazebo>
-      <link name="lpv_external_link"/>
-      <joint name="lpv_external_pivot_joint" type="universal">
-        <parent>lpv::lpv/base_link</parent>
-        <child>lpv_external_link</child>
-        <axis>
-          <xyz>1 0 0</xyz>
-        </axis>
-        <axis2>
-          <xyz>0 1 0</xyz>
-        </axis2>
-      </joint>
-      <joint name="lpv_external_riser" type="prismatic">
-        <parent>world</parent>
-        <child>lpv_external_link</child>
-        <axis>
-          <limit>
-            <lower>-3</lower>
-            <upper>3</upper>
-          </limit>
-          <xyz>0 0 1</xyz>
-        </axis>
-      </joint>
-    </gazebo>
-  </xacro:if>
   <!-- === Sensors === -->
   <!-- Use sensor yaml file if given -->
@@ -88,4 +68,7 @@
     <xacro:include filename="$(arg component_xacro_file)"/>
     <xacro:yaml_components />
+    <!-- Add CPU Cases -->
+    <xacro:include filename="$(find lpv_description)/urdf/cpu_cases.xacro" />
+    <xacro:cpu_cases position="-0.15 0 1.53" orientation="0 0 0"/>
   </xacro:if>
   <!-- Otherwise, add sensors based on enable variables -->
@@ -99,4 +82,12 @@
       <xacro:lpv_gps name="gps_lpv" x="-0.85" />
     </xacro:if>
+    <!-- Add Simulated IMU -->
+    <xacro:if value="$(arg imu_enabled)">
+      <xacro:lpv_imu name="imu_lpv" y="-0.2" />
+    </xacro:if>
+    <!-- Add 3D LIDAR -->
+    <xacro:if value="$(arg lidar_enabled)">
+      <xacro:lidar name="lidar_lpv" y="-0.3" type="16_beam"/>
+    </xacro:if>
     <!-- Add P3D ground truth -->
     <xacro:if value="$(arg ground_truth_enabled)">
@@ -107,12 +98,24 @@
       <xacro:lpv_pinger name="pinger" position="1.0 0 -1.0" />
     </xacro:if>
-    <!-- ==== AIMM sensor configuration ==== -->
+    <!-- Add ball shooter (default pitch angle: ~-60 deg) -->
+    <xacro:if value="$(arg ball_shooter_enabled)">
+      <xacro:lpv_ball_shooter name="ball_shooter" x="0.54" y="0.30" z="1.296" pitch="-1.04"/>
+    </xacro:if>
+    <!-- ==== LPV-4 sensor configuration ==== -->
     <xacro:if value="$(arg aimm_sensors_enabled)">
       <!-- Add a stereo camera pair -->
-      <xacro:lpv_camera name="front_left_camera" y="0.7" x="-3" z="0.9" P="${radians(0)}" Y="${radians(120)}" post_Y="${radians(120)}" visualize="true"/>
-      <xacro:lpv_camera name="front_right_camera" y="-0.7" x="-3" z="0.9" P="${radians(0)}" Y="${radians(-120)}" post_Y="${radians(-120)}" visualize="true"/>
-      <!-- Add simulated GPS + Radar -->
-      <xacro:lpv_gps name="gps_lpv" x="0.3" z="0.8"/>
-      <xacro:lpv_radar name="radar_lpv" x="-0.85" y="0" z="0.9" P="${radians(0)}" Y="${radians(-180)}"  />
+      <xacro:lpv_camera name="front_left_camera" y="0.4" x="2" z="0.5" P="${radians(0)}" Y="${radians(60)}" post_Y="${radians(120)}" visualize="true"/>
+      <xacro:lpv_camera name="front_right_camera" y="-0.4" x="2" z="0.5" P="${radians(0)}" Y="${radians(-60)}" post_Y="${radians(-120)}" visualize="true"/>
+      <!-- Add a camera facing right -->
+      <xacro:lpv_camera name="middle_rear_camera" x="-2" y="0" z="1" P="${radians(0)}" Y="${radians(180)}" post_Y="${radians(-120)}" visualize="true"/>
+      <!-- Add simulated GPS -->
+      <xacro:lpv_gps name="gps_lpv" x="-0.2" z="0.35" />
+      <!-- Add Simulated IMU -->
+      <xacro:lpv_imu name="imu_lpv" x="-0.2" y="0" z="0.35"/>
+      <!-- Add 3D LIDAR
+      <xacro:lidar name="lidar_lpv" type="16_beam"/>-->
+      <xacro:if value="$(arg ground_truth_enabled)">
+      <xacro:lpv_p3d name="p3d_lpv"/>
+    </xacro:if>
     </xacro:if>
   </xacro:unless>

File: lpv_gazebo/urdf/lpv_gazebo.xacro (robot description, xacro)
@@ -3,5 +3,5 @@
   <!-- Include macros for dynamics plugins -->
   <xacro:include filename="$(find lpv_gazebo)/urdf/macros.xacro" />
-  <!-- Macro to create a WAM-V with dyanmics plugins and a customizeable thruster layout -->
+  <!-- Macro to create a LPV-4 with dyanmics plugins and a customizeable thruster layout -->
   <xacro:macro  name="lpv_gazebo" params="thruster_layout">
     <!-- Defines the base vehicle -->

File: lpv_gazebo/urdf/macros.xacro (robot description, xacro)
@@ -2,5 +2,5 @@
 <!-- Includes all macros in this package so they don't need to be included individualy -->
 <robot xmlns:xacro="http://ros.org/wiki/xacro"
-       name="lpv-4">
+       name="LPV-4">
   <!-- Include dynamics macros -->
   <xacro:include filename="$(find lpv_gazebo)/urdf/dynamics/lpv_gazebo_dynamics_plugin.xacro" />
@@ -8,5 +8,4 @@
   <xacro:include filename="$(find lpv_gazebo)/urdf/components/lpv_camera.xacro" />
   <xacro:include filename="$(find lpv_gazebo)/urdf/components/lpv_gps.xacro" />
-  <xacro:include filename="$(find lpv_gazebo)/urdf/components/lpv_radar.xacro" />
   <xacro:include filename="$(find lpv_gazebo)/urdf/components/lpv_imu.xacro" />
   <xacro:include filename="$(find lpv_gazebo)/urdf/components/lpv_planar_lidar.xacro" />

File: lpv_gazebo/urdf/thruster_layouts/lpv_gazebo_thruster_config.xacro (robot description, xacro)
@@ -14,5 +14,5 @@
       <maxCmd>1.0</maxCmd>
       <maxForceFwd>250.0</maxForceFwd>
-      <maxForceRev>-250.0</maxForceRev>
+      <maxForceRev>-100.0</maxForceRev>
       <maxAngle>${pi/2}</maxAngle>
     </thruster>
